File: hw/backplane/backplane.kicad_pcb (KiCad board)
At the start: 2 copper layers, 26 parts, among them J1 out1, J10 conn5, J11 conn6, J12 out6, J2 out2, J3 conn2, J4 conn3, J5 conn1, J6 out3, J7 conn4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

Commit message: update backplane
Parts:
- added J13: Screw_Terminal_01x02, Connector_PinHeader_2.54mm:PinHeader_1x02_P2.54mm_Vertical, F.Cu at (61.0, 111.2)
- moved J12 140.8 mm to (261.3, 105.5), turned to 270 degrees
- moved J11 134.8 mm to (261.3, 117.5), turned to 270 degrees
- moved H14 132.4 mm to (267.6, 118.8)
- moved J9 123.9 mm to (225.4, 105.5), turned to 270 degrees
- moved H10 123.8 mm to (267.6, 106.8)
- moved J10 113.3 mm to (225.5, 117.4), turned to 270 degrees
- moved J8 100.6 mm to (189.6, 105.3), turned to 270 degrees
- moved H4 98.8 mm to (57.1, 118.6)
- moved H8 98.7 mm to (235.8, 106.8)
- moved H2 97.1 mm to (57.0, 106.4)
- moved J7 89.3 mm to (189.5, 117.4), turned to 270 degrees
- moved H1 87.4 mm to (235.8, 118.8)
- moved J6 76.4 mm to (153.7, 105.4), turned to 270 degrees
- moved H3 70.3 mm to (92.8, 106.5)
- moved J4 66.3 mm to (153.6, 117.3), turned to 270 degrees
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Connections:
- J1 pad 12: bus12 -> bus11
- J1 pad 14: bus14 -> bus13
- J10 pad 12: bus12 -> bus11
- J10 pad 14: bus14 -> bus13
- J11 pad 12: bus12 -> bus11
- J11 pad 14: bus14 -> bus13
- J11 pad 2: next_6 -> Net-(J11-Pad2)
- J12 pad 12: bus12 -> bus11
- J12 pad 14: bus14 -> bus13
- J2 pad 12: bus12 -> bus11
- J2 pad 14: bus14 -> bus13
- J3 pad 12: bus12 -> bus11
- J3 pad 14: bus14 -> bus13
- J4 pad 12: bus12 -> bus11
- J4 pad 14: bus14 -> bus13
- J5 pad 12: bus12 -> bus11
- J5 pad 14: bus14 -> bus13
- J5 pad 3: next_6 -> Net-(J5-Pad3)
- J6 pad 12: bus12 -> bus11
- J6 pad 14: bus14 -> bus13
- J7 pad 12: bus12 -> bus11
- J7 pad 14: bus14 -> bus13
- J8 pad 12: bus12 -> bus11
- J8 pad 14: bus14 -> bus13
- J9 pad 12: bus12 -> bus11
- J9 pad 14: bus14 -> bus13
Routing:
- net bus1: track 0.00 -> 294.2 mm
- net bus4: track 0.00 -> 288.6 mm
- net bus6: track 0.00 -> 287.6 mm
- net bus9: track 0.00 -> 287.1 mm
- net bus5: track 0.00 -> 287.0 mm
- net bus8: track 0.00 -> 287.0 mm
- net bus7: track 0.00 -> 286.9 mm
- net bus10: track 0.00 -> 286.9 mm
- net bus2: track 0.00 -> 218.4 mm
- net bus3: track 0.00 -> 188.6 mm
- net next_1: track 0.00 -> 95.4 mm, vias 0 -> 1
- net bus11: track 0.00 -> 84.7 mm
- net bus13: track 0.00 -> 84.7 mm
- net next_3: track 0.00 -> 55.6 mm, vias 0 -> 1
- net next_2: track 0.00 -> 54.7 mm, vias 0 -> 1
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- added copper zone on F.Cu, net bus11
- added copper zone on B.Cu, net bus13
Other:
- board outline added: 219.2 x 20.9 mm
- board text added: "5v"
- board text added: "GND"

Commit message: updates
Other:
- board text added: "Bricks"
- board text added: "I/O"
