File: hw/count/count.sch (KiCad schematic (older format))
At the start: 22 parts, among them J1 conn_trigger, J2 conn_done, J3 FTDI, J4 Conn_01x01_Male, J5 Conn_01x01_Male, J6 Conn_01x01_Male, J7 Conn_01x01_Male, SW1 reset_count, SW3 switch_reset, U1 ATmega328P-PU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

Commit message: update hardware
Parts:
- removed J4, J5, J6, J7: Conn_01x01_Male, Connector_PinHeader_2.54mm:PinHeader_1x01_P2.54mm_Vertical, symbol Connector:Conn_01x01_Male
Connections:
- wire segments 120 -> 97
- no-connect marks 0 -> 12
Changed lines of the file:
@@
 Wire Wire Line
 	10200 5400 10450 5400
-$Comp
-L Switch:SW_Push_Dual SW3
-U 1 1 5BD55A24
-P 4500 2700
-F 0 "SW3" H 4500 2985 50  0000 C CNN
-F 1 "switch_reset" H 4500 2894 50  0000 C CNN
-F 2 "autoblocks:SW_PUSH_6mm_H5mm" H 4500 2900 50  0001 C CNN
-F 3 "" H 4500 2900 50  0001 C CNN
-	1    4500 2700
-	1    0    0    -1
-$EndComp
 Wire Wire Line
 	4700 2700 4850 2700
@@
 	3100 2200 3200 2200
 Wire Wire Line
-	4250 2900 4250 3000
-Wire Wire Line
-	4250 3000 4750 3000
-Wire Wire Line
-	4300 2900 4250 2900
-Wire Wire Line
-	4700 2900 4750 2900
-Wire Wire Line
-	4750 2900 4750 3000
-Wire Wire Line
 	3100 2000 3200 2000
 Wire Wire Line
@@
 	1    0    0    -1
 $EndComp
-$Comp
-L Switch:SW_Push_Dual SW1
-U 1 1 5BC62516
-P 9250 1850
-F 0 "SW1" H 9250 2135 50  0000 C CNN
-F 1 "reset_count" H 9250 2044 50  0000 C CNN
-F 2 "autoblocks:SW_PUSH_6mm_H5mm" H 9250 2050 50  0001 C CNN
-F 3 "" H 9250 2050 50  0001 C CNN
-	1    9250 1850
-	1    0    0    -1
-$EndComp
 Text GLabel 6700 3550 0    50   Input ~ 0
 a3
@@
 Wire Wire Line
 	9450 1850 9700 1850
-Wire Wire Line
-	9050 2050 8950 2050
-Wire Wire Line
-	8950 2050 8950 2150
-Wire Wire Line
-	8950 2150 9550 2150
-Wire Wire Line
-	9550 2150 9550 2050
-Wire Wire Line
-	9550 2050 9450 2050
-Wire Wire Line
-	850  5950 850  6000
-Wire Wire Line
-	850  6000 1150 6000
-Wire Wire Line
-	1150 6000 1150 5950
-Wire Wire Line
-	1150 6000 1250 6000
-Wire Wire Line
-	1400 6000 1400 5950
-Connection ~ 1150 6000
-Wire Wire Line
-	1400 6000 1650 6000
-Wire Wire Line
-	1650 6000 1650 5950
-Connection ~ 1400 6000
-$Comp
-L power:GND #PWR0102
-U 1 1 5BC936D3
-P 1250 6100
-F 0 "#PWR0102" H 1250 5850 50  0001 C CNN
-F 1 "GND" H 1255 5927 50  0000 C CNN
-F 2 "" H 1250 6100 50  0001 C CNN
-F 3 "" H 1250 6100 50  0001 C CNN
-	1    1250 6100
-	1    0    0    -1
-$EndComp
-Wire Wire Line
-	1250 6100 1250 6000
-Connection ~ 1250 6000
-Wire Wire Line
-	1250 6000 1400 6000
-$Comp
-L Connector:Conn_01x01_Male J4
-U 1 1 5BC9D551
-P 7150 4000
-F 0 "J4" H 7050 4000 50  0000 C CNN
-F 1 "Conn_01x01_Male" H 6650 4000 50  0000 C CNN
-F 2 "Connector_PinHeader_2.54mm:PinHeader_1x01_P2.54mm_Vertical" H 7150 4000 50  0001 C CNN
-F 3 "~" H 7150 4000 50  0001 C CNN
-	1    7150 4000
-	-1   0    0    1
-$EndComp
 Text GLabel 6700 4000 0    50   Input ~ 0
 d9
@@
 a2
 $Comp
-L Connector:Conn_01x01_Male J5
-U 1 1 5BCACA1A
-P 7150 4150
-F 0 "J5" H 7050 4150 50  0000 C CNN
-F 1 "Conn_01x01_Male" H 6650 4150 50  0000 C CNN
-F 2 "Connector_PinHeader_2.54mm:PinHeader_1x01_P2.54mm_Vertical" H 7150 4150 50  0001 C CNN
-F 3 "~" H 7150 4150 50  0001 C CNN
-	1    7150 4150
-	-1   0    0    1
-$EndComp
-$Comp
-L Connector:Conn_01x01_Male J6
-U 1 1 5BCACA54
-P 7150 4300
-F 0 "J6" H 7050 4300 50  0000 C CNN
-F 1 "Conn_01x01_Male" H 6650 4300 50  0000 C CNN
-F 2 "Connector_PinHeader_2.54mm:PinHeader_1x01_P2.54mm_Vertical" H 7150 4300 50  0001 C CNN
-F 3 "~" H 7150 4300 50  0001 C CNN
-	1    7150 4300
-	-1   0    0    1
-$EndComp
-$Comp
-L Connector:Conn_01x01_Male J7
-U 1 1 5BCACA8E
-P 7150 4450
-F 0 "J7" H 7050 4450 50  0000 C CNN
-F 1 "Conn_01x01_Male" H 6650 4450 50  0000 C CNN
-F 2 "Connector_PinHeader_2.54mm:PinHeader_1x01_P2.54mm_Vertical" H 7150 4450 50  0001 C CNN
-F 3 "~" H 7150 4450 50  0001 C CNN
-	1    7150 4450
-	-1   0    0    1
-$EndComp
-Wire Wire Line
-	6700 4000 6950 4000
-Wire Wire Line
-	6700 4150 6950 4150
-Wire Wire Line
-	6700 4300 6950 4300
-Wire Wire Line
-	6700 4450 6950 4450
+L Switch:SW_Push_Dual SW1
+U 1 1 5BC62516
+P 9250 1850
+F 0 "SW1" H 9250 2135 50  0000 C CNN
+F 1 "reset_count" H 9250 2044 50  0000 C CNN
+F 2 "autoblocks:SW_PUSH_6mm_H5mm" H 9250 2050 50  0001 C CNN
+F 3 "" H 9250 2050 50  0001 C CNN
+	1    9250 1850
+	1    0    0    -1
+$EndComp
+NoConn ~ 9450 2050
+NoConn ~ 9050 2050
+$Comp
+L Switch:SW_Push_Dual SW3
+U 1 1 5BD55A24
+P 4500 2700
+F 0 "SW3" H 4500 2985 50  0000 C CNN
+F 1 "switch_reset" H 4500 2894 50  0000 C CNN
+F 2 "autoblocks:SW_PUSH_6mm_H5mm" H 4500 2900 50  0001 C CNN
+F 3 "" H 4500 2900 50  0001 C CNN
+	1    4500 2700
+	1    0    0    -1
+$EndComp
+NoConn ~ 4700 2900
+NoConn ~ 4300 2900
+NoConn ~ 850  5950
+NoConn ~ 1150 5950
+NoConn ~ 1400 5950
+NoConn ~ 1650 5950
+NoConn ~ 6700 4000
+NoConn ~ 6700 4150
+NoConn ~ 6700 4300
+NoConn ~ 6700 4450
 $EndSCHEMATC

Commit message: COUNT block v2
Parts:
- removed J1: conn_trigger, Connector_PinHeader_2.54mm:PinHeader_1x03_P2.54mm_Vertical, symbol Connector:Conn_01x03_Male
- removed J2: conn_done, Connector_PinHeader_2.54mm:PinHeader_1x03_P2.54mm_Vertical, symbol Connector:Conn_01x03_Male
- removed SW1: reset_count, autoblocks:SW_PUSH_6mm_H5mm, symbol Switch:SW_Push_Dual
- removed SW3: switch_reset, autoblocks:SW_PUSH_6mm_H5mm, symbol Switch:SW_Push_Dual
- removed U1: ATmega328P-PU, Package_DIP:DIP-28_W7.62mm, symbol MCU_Microchip_ATmega:ATmega328P-PU
- added J1: bootloader, autoblocks:edge_connector_3, symbol Connector:Conn_01x06_Male
- added J5: BUS, Connector_PinHeader_2.54mm:PinHeader_2x07_P2.54mm_Vertical, symbol Connector_Generic:Conn_02x07_Counter_Clockwise
- added R5, R6, R7: 1k, Resistor_SMD:R_0603_1608Metric, symbol Device:R
- added SW2: resetCount, autoblocks:SW_PUSH_6mm_H5mm, symbol Switch:SW_Push
- added SW3: reset, Button_Switch_SMD:SW_SPST_TL3305C, symbol Switch:SW_Push
- added SW4: NEXT, Package_DIP:DIP-16_W7.62mm_SMDSocket_SmallPads, symbol Switch:SW_DIP_x08
- added SW6: ID, Package_DIP:DIP-16_W7.62mm_SMDSocket_SmallPads, symbol Switch:SW_DIP_x08
- added U1: ATmega328-AU, Package_QFP:TQFP-32_7x7mm_P0.8mm, symbol MCU_Microchip_ATmega:ATmega328-AU
- C1: footprint Capacitor_THT:CP_Radial_Tantal_D6.0mm_P2.50mm -> Capacitor_SMD:C_0603_1608Metric
- C2, C3: footprint Capacitor_THT:C_Disc_D3.0mm_W1.6mm_P2.50mm -> Capacitor_SMD:C_0603_1608Metric
- C4, C5: footprint Capacitor_THT:C_Axial_L5.1mm_D3.1mm_P7.50mm_Horizontal -> Capacitor_SMD:C_0603_1608Metric
- H1, H2, H3, H4: footprint MountingHole:MountingHole_2.2mm_M2 -> MountingHole:MountingHole_3.2mm_M3_Pad
- J3: footprint Connector_PinHeader_2.54mm:PinHeader_1x06_P2.54mm_Vertical -> autoblocks:edge_connector_3
- R2: footprint Resistor_THT:R_Axial_DIN0207_L6.3mm_D2.5mm_P10.16mm_Horizontal -> Resistor_SMD:R_0603_1608Metric
- Y1: footprint Crystal:Crystal_HC18-U_Vertical -> Crystal:Crystal_SMD_HC49-SD
Connections:
- net AREF: now also U1.20 (AREF)
- net GND: now also J1.1 (Pin_1), J5.13 (Pin_13), J5.14 (Pin_14), SW2.2, SW3.1, U1.21 (GND), U1.3 (GND), U1.5 (GND)
- net RESET: now also SW3.2, U1.29 (~RESET~/PC6)
- net RX: now also J5.9 (Pin_9), U1.30 (PD0)
- net TX: now also J5.10 (Pin_10), U1.31 (PD1)
- net VCC: now also J1.2 (Pin_2), J5.11 (Pin_11), J5.12 (Pin_12), U1.18 (AVCC), U1.4 (VCC), U1.6 (VCC)
- net XTAL1: now also U1.7 (XTAL1/PB6)
- net XTAL2: now also U1.8 (XTAL2/PB7)
- net a0: now also SW6.1, SW6.2, SW6.3, SW6.4, SW6.5, SW6.6, SW6.7, SW6.8, U1.23 (PC0)
- net a1: now also SW4.10, SW4.11, SW4.12, SW4.13, SW4.14, SW4.15, SW4.16, SW4.9, U1.24 (PC1)
- net a2: now also U1.25 (PC2)
- net a3: now also SW2.1, U1.26 (PC3)
- net a4: now also R6.1, U1.27 (PC4); no longer U2.5 (cc2)
- net a5: now also R7.1, U1.28 (PC5); no longer U2.7 (cc3)
- net d10: now also J1.3 (Pin_3), U1.14 (PB2)
- net d11: now also J1.4 (Pin_4), U1.15 (PB3)
- net d12: now also J1.5 (Pin_5), U1.16 (PB4)
- net d13: now also J1.6 (Pin_6), R5.1, U1.17 (PB5); no longer U2.1 (cc1)
- net d2: now also U1.32 (PD2)
- net d3: now also U1.1 (PD3)
- net d4: now also U1.2 (PD4)
- net d5: now also U1.9 (PD5)
- net d6: now also U1.10 (PD6)
- net d7: now also U1.11 (PD7)
- net d8: now also U1.12 (PB0)
- net d9: now also U1.13 (PB1)
- new net: R5.2, U2.1 (cc1)
- new net: R6.2, U2.5 (cc2)
- new net: R7.2, U2.7 (cc3)
- new net bus1: J5.1 (Pin_1), SW4.1, SW6.9
- new net bus2: J5.2 (Pin_2), SW4.2, SW6.10
- new net bus3: J5.3 (Pin_3), SW4.3, SW6.11
- new net bus4: J5.4 (Pin_4), SW4.4, SW6.12
- new net bus5: J5.5 (Pin_5), SW4.5, SW6.13
- new net bus6: J5.6 (Pin_6), SW4.6, SW6.14
- new net bus7: J5.7 (Pin_7), SW4.7, SW6.15
- new net bus8: J5.8 (Pin_8), SW4.8, SW6.16
- no-connect marks 12 -> 8
Other:
- moved on the sheet: J3, U2

Commit message: fix COUNT bus assigments
Connections:
- net a0: now also SW6.10, SW6.11, SW6.12, SW6.13, SW6.14, SW6.15, SW6.16, SW6.9; no longer SW6.1, SW6.2, SW6.3, SW6.4, SW6.5, SW6.6, SW6.7, SW6.8
- net bus1: now also SW6.1; no longer SW6.9
- net bus2: now also SW6.2; no longer SW6.10
- net bus3: now also SW6.3; no longer SW6.11
- net bus4: now also SW6.4; no longer SW6.12
- net bus5: now also SW6.5; no longer SW6.13
- net bus6: now also SW6.6; no longer SW6.14
- net bus7: now also SW6.7; no longer SW6.15
- net bus8: now also SW6.8; no longer SW6.16
Changed lines of the file:
@@
 L Switch:SW_DIP_x08 SW6
 U 1 1 5C35B265
-P 7550 1500
-F 0 "SW6" H 7550 900 50  0000 C CNN
-F 1 "ID" H 7550 1000 50  0000 C CNN
-F 2 "Package_DIP:DIP-16_W7.62mm_SMDSocket_SmallPads" H 7550 1500 50  0001 C CNN
-F 3 "" H 7550 1500 50  0001 C CNN
-	1    7550 1500
-	-1   0    0    1
+P 7550 1600
+F 0 "SW6" H 7550 1000 50  0000 C CNN
+F 1 "ID" H 7550 1100 50  0000 C CNN
+F 2 "Package_DIP:DIP-16_W7.62mm_SMDSocket_SmallPads" H 7550 1600 50  0001 C CNN
+F 3 "" H 7550 1600 50  0001 C CNN
+	1    7550 1600
+	1    0    0    -1
 $EndComp
 $Comp
